Commit message: 

File: protomotions/data/assets/urdf/go2.urdf (robot description, URDF)
Before this commit: robot go2, 41 links, 40 joints
Links:
- link base: geometry collision box size=0.3762 0.0935 0.114; visual mesh filename=../mesh/go2/base.dae

Commit message: 

File: protomotions/data/assets/urdf/go2.urdf (robot description, URDF)
Before this commit: robot go2, 41 links, 40 joints
Links:
- removed link Head_lower
- removed link Head_upper
Joints:
- removed joint Head_lower_joint
- removed joint Head_upper_joint
